File: 208_Timbre_Workshop_Panel.kicad_pcb (KiCad board)
At the start: 2 copper layers, 40.3 x 128.5 mm, 2 parts

Commit message: alignment, transistor pins
Routing:
- added copper zone on F.Cu, net (none)
Changed lines of the file:
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@@
   (gr_curve (pts (xy 149.400003 100.6) (xy 150.155411 100.6) (xy 150.767791 99.98762) (xy 150.767791 99.232212))
     (stroke (width 0.05) (type solid)) (layer "Edge.Cuts"))
-  (zone (net 0) (net_name "") (layer "B.Cu") (hatch edge 0.5)
+  (zone (net 0) (net_name "") (layers "F&B.Cu") (hatch edge 0.5)
     (connect_pads (clearance 0.508))
     (min_thickness 0.25) (filled_areas_thickness no)
