File: 208_Timbre_Workshop.kicad_sch (KiCad schematic)
At the start: 79 parts, among them J1 CV_IN, J2 AUDIO_IN, J3 AUDIO_OUT, J4 30310-6002HB, J5 Conn_01x05_Female, J6 Conn_01x05_Male, Q5 2N3905, Q6 J201, U1 TL072, U2 TL074, U3 TL074

Commit message: alignment, transistor pins
Parts:
- removed Q5: 2N3905, Triglav_Modular:TO-92, symbol Device:Q_PNP_BCE
- added Q5: 2N3905, Triglav_Modular:TO-92, symbol Device:Q_PNP_EBC
- CX6: value 50n -> 47n*
Connections:
- net GND: now also Q6.2 (D), Q5.2 (B); no longer Q6.1 (S)
- net at C1.1, R24.1, VR1.1: now also Q5.3 (C)
- net at C2.2, R21.1: now also Q6.1 (S); no longer Q6.2 (D)
- net at R23.1: now also Q5.1 (E)
Changed lines of the file:
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@@
+    )
+  )
+  (symbol (lib_id "Device:Q_PNP_EBC") (at 104.14 151.13 270) (mirror x) (unit 1)
+    (in_bom yes) (on_board yes) (dnp no) (fields_autoplaced)
+    (property "Reference" "Q5" (at 104.14 143.51 90)
+      (effects (font (size 1.27 1.27)))
+    )
+    (property "Value" "2N3905" (at 104.14 146.05 90)
+      (effects (font (size 1.27 1.27)))
+    )
+    (property "Footprint" "Triglav_Modular:TO-92" (at 106.68 146.05 0)
+      (effects (font (size 1.27 1.27)) hide)
+    )
+    (property "Datasheet" "~" (at 104.14 151.13 0)
+      (effects (font (size 1.27 1.27)) hide)
+    )
+    (pin "1")
+    (pin "2")
+    (pin "3")
+    (instances
+      (project "208_Timbre_Workshop"
+        (path "/01c2f37b-a975-4458-92af-15e8e08e5f2e"
+          (reference "Q5") (unit 1)
+        )
+      )
     )
   )
@@
     )
   )
-  (symbol (lib_id "Device:Q_NJFET_SDG") (at 152.4 118.11 0) (unit 1)
-    (in_bom yes) (on_board yes) (dnp no) (fields_autoplaced)
-    (property "Reference" "Q6" (at 157.48 116.8399 0)
-      (effects (font (size 1.27 1.27)) (justify left))
-    )
-    (property "Value" "J201" (at 157.48 119.3799 0)
-      (effects (font (size 1.27 1.27)) (justify left))
-    )
-    (property "Footprint" "Triglav_Modular:TO-92" (at 157.48 115.57 0)
+  (symbol (lib_id "Device:Q_NJFET_SDG") (at 152.4 118.11 0) (mirror x) (unit 1)
+    (in_bom yes) (on_board yes) (dnp no)
+    (property "Reference" "Q6" (at 157.48 119.3801 0)
+      (effects (font (size 1.27 1.27)) (justify left))
+    )
+    (property "Value" "J201" (at 157.48 116.8401 0)
+      (effects (font (size 1.27 1.27)) (justify left))
+    )
+    (property "Footprint" "Triglav_Modular:TO-92" (at 157.48 120.65 0)
       (effects (font (size 1.27 1.27)) hide)
     )
@@
   (symbol (lib_id "Device:C") (at 78.74 245.11 0) (mirror x) (unit 1)
     (in_bom yes) (on_board yes) (dnp no) (fields_autoplaced)
-    (property "Reference" "CX6" (at 74.93 243.8399 0)
-      (effects (font (size 1.27 1.27)) (justify right))
-    )
-    (property "Value" "50n" (at 74.93 246.3799 0)
+    (property "Reference" "CX6" (at 74.93 244.475 0)
+      (effects (font (size 1.27 1.27)) (justify right))
+    )
+    (property "Value" "47n*" (at 74.93 247.015 0)
       (effects (font (size 1.27 1.27)) (justify right))
     )
@@
         )
       )
-    )
-  )
-  (symbol (lib_id "Device:Q_PNP_BCE") (at 104.14 151.13 270) (mirror x) (unit 1)
-    (in_bom yes) (on_board yes) (dnp no) (fields_autoplaced)
-    (property "Reference" "Q5" (at 104.14 142.24 90)
-      (effects (font (size 1.27 1.27)))
-    )
-    (property "Value" "2N3905" (at 104.14 144.78 90)
-      (effects (font (size 1.27 1.27)))
-    )
-    (property "Footprint" "Triglav_Modular:TO-92" (at 106.68 146.05 0)
-      (effects (font (size 1.27 1.27)) hide)
-    )
-    (property "Datasheet" "~" (at 104.14 151.13 0)
-      (effects (font (size 1.27 1.27)) hide)
-    )
-    (pin "1")
-    (pin "2")
-    (pin "3")
-    (instances
-      (project "208_Timbre_Workshop"
-        (path "/01c2f37b-a975-4458-92af-15e8e08e5f2e"
-          (reference "Q5") (unit 1)
-        )
-      )

Commit message: Cleanup
Parts:
- Q6: value J201 -> 2N4341; footprint Triglav_Modular:TO-92 -> Triglav_Modular:TO-18-3
- RX1: value 10k -> 68k
- U1: value TL072 -> TL072*
- U2, U3: value TL074 -> TL084*
- VR1: Silkscreen_Name CV Gain -> Control Gain
- VRX1: Silkscreen_Name Input volume -> Input Volume
Connections:
- net pin3: now reaches Q6.3 (G), R18.2, R22.1
Other:
- moved on the sheet: J5, J6, R21

Commit message: Cleanup
Parts:
- RX1: value 68k -> 10k
- RX3: value 10k -> 3k3
Changed lines of the file:
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@@
       (effects (font (size 1.27 1.27)) (justify right))
     )
-    (property "Value" "10k" (at 308.61 73.025 0)
+    (property "Value" "3k3" (at 308.61 73.025 0)
       (effects (font (size 1.27 1.27)) (justify right))
     )
@@
       (effects (font (size 1.27 1.27)))
     )
-    (property "Value" "68k" (at 312.42 82.55 90)
-      (effects (font (size 1.27 1.27)))
-    )
+    (property "Value" "10k" (at 312.42 82.55 90)
+      (effects (font (size 1.27 1.27)))
+    )

Commit message: Cleanup
Connections:
- net at R37.2, R38.1, R42.2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: now also R43.2; no longer R43.1
- net at R38.2, R39.1, R45.2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: now also R43.1; no longer R43.2
- net NI_GND1 renamed GND2
- net NI_GND2 renamed GND3
Other:
- note added: "(44k2)"
- note added: "(71k4)"
- moved on the sheet: R29, R33, R36, R38, R43, R47

Commit message: Cleanup
Connections:
- net GND: no longer J1.S, J2.S, J3.S, J5.2 (Pin_2), VR2.1, VR3.1
- net +15V renamed +12V
- net -15V renamed -12V
- net pin3: no longer names the net of Q6.3 (G), R18.2, R22.1
- new net P_GND: J1.S, J2.S, J3.S, J5.2 (Pin_2), VR2.1, VR3.1
Other:
- note added: "CV slider"
- note added: "Timbre slider"
- note removed: "CV"
- note removed: "Timbre"
- moved on the sheet: C10, C11, C4, C5, C6, C7, C8, C9, CX5, CX6, D3, D4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
