File: 208_Timbre_Workshop.kicad_sch (KiCad schematic)
At the start: 79 parts, among them J1 CV_IN, J2 AUDIO_IN, J3 AUDIO_OUT, J4 30310-6002HB, J5 Conn_01x05_Female, J6 Conn_01x05_Male, Q5 2N3905, Q6 2N4341, U1 TL072*, U2 TL084*, U3 TL084*

Commit message: transistor update
Connections:
- net GND: now also Q6.1 (S); no longer Q6.2 (D)
- net at C2.2, R21.1: now also Q6.2 (D); no longer Q6.1 (S)
Changed lines of the file:
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@@
     )
   )
-  (symbol (lib_id "Device:Q_NJFET_SDG") (at 152.4 118.11 0) (mirror x) (unit 1)
+  (symbol (lib_id "Device:Q_NJFET_SDG") (at 152.4 118.11 0) (unit 1)
     (in_bom yes) (on_board yes) (dnp no)
-    (property "Reference" "Q6" (at 157.48 119.3801 0)
+    (property "Reference" "Q6" (at 157.48 116.8399 0)
       (effects (font (size 1.27 1.27)) (justify left))
     )
-    (property "Value" "2N4341" (at 157.48 116.8401 0)
+    (property "Value" "2N4341" (at 157.48 119.3799 0)
       (effects (font (size 1.27 1.27)) (justify left))
     )
-    (property "Footprint" "Triglav_Modular:TO-18-3" (at 157.48 120.65 0)
+    (property "Footprint" "Triglav_Modular:TO-18-3" (at 157.48 115.57 0)
       (effects (font (size 1.27 1.27)) hide)
     )

Commit message: Rev. 2
Parts:
- C2: value 15uF -> 15u
- D3, D4: value 1N5819 -> 1N5817
- U2, U3: value TL084* -> RC4136; symbol Amplifier_Operational:TL074 -> Triglav_Modular:RC4136
Connections:
- net P_GND is gone; now on net GND: J1.S, J2.S, J3.S, J5.2 (Pin_2), VR2.1, VR3.1
- net +12V: now also U2.11 (V+), U3.11 (V+); no longer U2.4 (V+), U3.4 (V+)
- net -12V: now also U2.7 (V-), U3.7 (V-); no longer U2.11 (V-), U3.11 (V-)
- net GND2: now also U2.2 (+), U2.9 (+), U3.13 (+); no longer U2.10 (+), U2.3 (+), U3.12 (+)
- net GND3: now also U3.2 (+), U3.9 (+); no longer U3.10 (+), U3.3 (+)
- net at C3.1, D1.1 (K), D2.2 (A)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: now also U2.8 (-); no longer U2.9 (-)
- net at C3.2, D1.2 (A), D2.1 (K)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: now also U2.10; no longer U2.8
- net at R32.1: now also U2.4; no longer U2.7
- net at U2.1 (-): now also R25.1, R26.2, R27.2; no longer R27.1
- net at R1.2, R18.1, R19.1: now also U2.13 (+); no longer U2.12 (+)
- net at C2.1, R20.1: now also U2.14 (-); no longer U2.13 (-)
- net at R20.2, R25.2, R28.2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: now also U2.12; no longer U2.14
- net at R42.1: now also U3.4; no longer U3.7
- net at R39.2, R40.1: now also U3.10; no longer U3.8
- net at U3.1 (-): now also R41.2, R44.2, R45.1; no longer R44.1
- net at R38.2, R39.1, R43.1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: now also U3.8 (-); no longer U3.9 (-)
- net at R34.1: now also U3.12; no longer U3.14
- net at R31.1, R34.2, R35.1: now also U3.14 (-); no longer U3.13 (-)
- new net: R27.1, U2.3
- new net: R44.1, U3.3

Commit message: Rev.2
Other:
- title: Buchla 208 Timbre (ASS Edition) -> 208 Timbre 
Changed lines of the file:
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@@
   (paper "A3")
   (title_block
-    (title "Buchla 208 Timbre (ASS Edition)")
-    (date "2023-04-26")
-    (rev "1")
+    (title "208 Timbre ")
+    (date "2023-07-29")
+    (rev "2")
     (company "Triglav Modular")
     (comment 1 "1975")
