File: 208_Timbre_Workshop.kicad_pcb (KiCad board)
At the start: 2 copper layers, 80.5 x 113 mm, 93 parts, among them J1 CV_IN, J2 AUDIO_IN, J3 AUDIO_OUT, J4 30310-6002HB, J5 Conn_01x05_Female, J6 Conn_01x05_Male, Q5 2N3905, Q6 J201, U1 TL072, U2 TL074, U3 TL074

Commit message: alignment, transistor pins
Parts:
- CX6: value 50n -> 47n*
- moved D4 3.10 mm to (167.6, 147.4)
- moved VR2 0.38 mm to (144.7, 78.5)
- moved VR3 0.38 mm to (124.1, 78.5)
- moved RX1 0.12 mm to (163.8, 118.6)
Connections:
- C2 pad 2: Net-(Q6-D) -> Net-(Q6-S)
- Q5 pad 1: P_GND -> Net-(Q5-E)
- Q5 pad 2: Net-(Q5-C) -> P_GND
- Q5 pad 3: Net-(Q5-E) -> Net-(Q5-C)
- Q6 pad 1: P_GND -> Net-(Q6-S)
- Q6 pad 2: Net-(Q6-D) -> P_GND
- R21 pad 1: Net-(Q6-D) -> Net-(Q6-S)
Routing:
- net Net-(Q6-S): track 0.00 -> 21.3 mm
- net Net-(Q6-D): track 20.3 -> 0.00 mm
- net Net-(D4-K): track 28.3 -> 25.2 mm
- net Net-(Q5-E): track 6.79 -> 9.33 mm
- net Net-(Q5-C): track 20.5 -> 22.3 mm
- net VREF: track 68.3 -> 67.2 mm
- net -15V: track 138.1 -> 137.2 mm
- net +15V: track 128.2 -> 128.8 mm

Commit message: Cleanup
Parts:
- removed the REF** at (191.7, 46.0)
- removed the REF** at (157.5, 152.9)
- removed the REF** at (117.2, 152.9)
- removed the REF** at (151.5, 46.0)
- Q6: value J201 -> 2N4341; footprint Triglav_Modular:TO-92 -> Triglav_Modular:TO-18-3
- RX1: value 10k -> 68k
- U1: value TL072 -> TL072*
- U2, U3: value TL074 -> TL084*
- moved REF** 29.6 mm to (184.6, 57.9)
- moved REF** 20.9 mm to (134.4, 57.9)
- moved G*** 20.7 mm to (90.0, 135.0)
- moved REF** 17.4 mm to (134.4, 149.8)
- moved G*** 16.8 mm to (208.6, 149.0)
- moved Q6 16.1 mm to (193.7, 56.5), turned to 180 degrees
- moved VRX1 14.3 mm to (199.7, 54.1)
- moved C1 13.6 mm to (187.8, 51.8)
- moved R24 12.5 mm to (190.1, 47.2)
- moved R22 12.4 mm to (179.7, 47.2)
- moved C2 11.7 mm to (181.3, 51.9)
- moved C7 11.5 mm to (177.8, 123.7)
- moved C6 11.1 mm to (172.4, 71.7)
- moved VR1 10.1 mm to (175.4, 54.1)
- moved C10 10.0 mm to (174.0, 143.0)
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Connections:
- net Net-(Q6-G) renamed /pin3
Routing:
- net Net-(Q5-C): track 22.3 -> 28.7 mm
- net M_Audio_In: track 106.9 -> 111.1 mm
- net P_GND: track 0.00 -> 3.63 mm
- net -15V: track 137.2 -> 140.6 mm
- net Net-(Q6-S): track 21.3 -> 23.9 mm
- net /pin3: track 33.8 -> 36.3 mm
- net Net-(R1-Pad1): track 25.2 -> 23.0 mm
- net Net-(U2D-+): track 15.9 -> 13.9 mm
- net +15V: track 128.8 -> 127.4 mm
- net Net-(U2D--): track 32.4 -> 33.7 mm
- net Net-(D4-K): track 25.2 -> 24.0 mm
- net VREF: track 67.2 -> 66.0 mm
- net Net-(R22-Pad2): track 6.40 -> 7.14 mm
- net Net-(QX2-B): track 16.7 -> 16.2 mm
- net Net-(R39-Pad2): track 42.2 -> 42.4 mm, vias 1 -> 0
Other:
- board size 80.5 x 113 mm -> 90.5 x 108.9 mm

Commit message: Cleanup
Parts:
- RX1: value 68k -> 10k
- RX3: value 10k -> 3k3
Changed lines of the file:
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@@
         (effects (font (size 1 1) (thickness 0.15)))
     )
-    (fp_text value "10k" (at -0.0216 0.124975) (layer "F.SilkS")
+    (fp_text value "3k3" (at -0.0216 0.124975) (layer "F.SilkS")
         (effects (font (size 1 1) (thickness 0.15)))
     )
@@
         (effects (font (size 1 1) (thickness 0.15)))
     )
-    (fp_text value "68k" (at -0.0216 0.124975) (layer "F.SilkS")
+    (fp_text value "10k" (at -0.0216 0.124975) (layer "F.SilkS")
         (effects (font (size 1 1) (thickness 0.15)))
     )

Commit message: Cleanup
Parts:
- turned R43 to 180 degrees
Connections:
- net +15V renamed +12V
- net -15V renamed -12V
- net /NI_GND1 renamed /GND2
- net /NI_GND2 renamed /GND3
- net /pin3 renamed Net-(Q6-G)
- C1 pad 2: P_GND -> GND
- C10 pad 2: P_GND -> GND
- C11 pad 1: P_GND -> GND
- C4 pad 1: P_GND -> GND
- C5 pad 2: P_GND -> GND
- C6 pad 1: P_GND -> GND
- C7 pad 2: P_GND -> GND
- C8 pad 1: P_GND -> GND
- C9 pad 2: P_GND -> GND
- J4 pad 3: P_GND -> GND
- J4 pad 4: P_GND -> GND
- J4 pad 5: P_GND -> GND
- J4 pad 6: P_GND -> GND
- J4 pad 7: P_GND -> GND
- J4 pad 8: P_GND -> GND
- J6 pad 2: P_GND -> GND
- Q5 pad 2: P_GND -> GND
- Q6 pad 2: P_GND -> GND
- R19 pad 2: P_GND -> GND
- R21 pad 2: P_GND -> GND
- R36 pad 2: P_GND -> GND
- R43 pad 1: Net-(U3B--) -> Net-(U3C--)
- R43 pad 2: Net-(U3C--) -> Net-(U3B--)
- R47 pad 2: P_GND -> GND
- RX3 pad 1: P_GND -> GND
- RX32 pad 1: P_GND -> GND
- RX52 pad 1: P_GND -> GND
- VR1 pad 3: P_GND -> GND
Routing:
- net P_GND: track 3.63 -> 0.00 mm
- net GND: track 0.00 -> 3.63 mm
- added copper zone on B.Cu, net GND
- added copper zone on F.Cu, net GND

Commit message: Cleanup
Parts:
- moved G*** 44.3 mm to (134.4, 135.0)

Commit message: transistor update
Connections:
- C2 pad 2: Net-(Q6-S) -> Net-(Q6-D)
- Q6 pad 1: Net-(Q6-S) -> GND
- Q6 pad 2: GND -> Net-(Q6-D)
- R21 pad 1: Net-(Q6-S) -> Net-(Q6-D)
Routing:
- net Net-(Q6-S): track 23.9 -> 0.00 mm
- net Net-(Q6-D): track 0.00 -> 22.8 mm
- net GND: track 3.63 -> 0.05 mm
Changed lines of the file:
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@@
   (net 1 "Net-(Q5-C)")
   (net 2 "Net-(U2D--)")
-  (net 3 "Net-(Q6-S)")
+  (net 3 "Net-(Q6-D)")
   (net 4 "Net-(D1-K)")
   (net 5 "Net-(D1-A)")
@@
       (net 2 "Net-(U2D--)") (pintype "passive"))
     (pad "2" thru_hole circle (at 2 0) (size 1.6 1.6) (drill 0.8) (layers "*.Cu" "*.Mask")
-      (net 3 "Net-(Q6-S)") (pintype "passive"))
+      (net 3 "Net-(Q6-D)") (pintype "passive"))
     (model "${KICAD6_3DMODEL_DIR}/Capacitor_THT.3dshapes/CP_Radial_D5.0mm_P2.00mm.wrl"
       (offset (xyz 0 0 0))
@@
       (stroke (width 0.1) (type solid)) (layer "F.Fab"))
     (pad "1" thru_hole circle (at -3.81 0 270) (size 1.6 1.6) (drill 0.8) (layers "*.Cu" "*.Mask")
-      (net 3 "Net-(Q6-S)") (pintype "passive"))
+      (net 3 "Net-(Q6-D)") (pintype "passive"))
     (pad "2" thru_hole oval (at 3.81 0 270) (size 1.6 1.6) (drill 0.8) (layers "*.Cu" "*.Mask")
       (net 6 "GND") (pintype "passive"))
@@
       (stroke (width 0.1) (type solid)) (fill none) (layer "F.Fab"))
     (pad "1" thru_hole oval (at 0 0 225) (size 1.6 1.2) (drill 0.7) (layers "*.Cu" "*.Mask")
-      (net 3 "Net-(Q6-S)") (pinfunction "S") (pintype "passive"))
+      (net 6 "GND") (pinfunction "S") (pintype "passive"))
     (pad "2" thru_hole oval (at 1.27 1.27 180) (size 1.2 1.2) (drill 0.7) (layers "*.Cu" "*.Mask")
-      (net 6 "GND") (pinfunction "D") (pintype "passive"))
+      (net 3 "Net-(Q6-D)") (pinfunction "D") (pintype "passive"))
     (pad "3" thru_hole oval (at 2.54 0 180) (size 1.2 1.2) (drill 0.7) (layers "*.Cu" "*.Mask")
       (net 23 "Net-(Q6-G)") (pinfunction "G") (pintype "input"))
@@
   (segment (start 183.91005 63.62325) (end 183.91005 65.510425) (width 0.5) (layer "B.Cu") (net 2))
   (segment (start 181.3484 51.8922) (end 181.3484 61.0616) (width 0.5) (layer "B.Cu") (net 2))
-  (segment (start 193.6774 56.55) (end 193.6274 56.55) (width 0.5) (layer "F.Cu") (net 3))
-  (segment (start 193.6274 56.55) (end 192.3076 57.8698) (width 0.5) (layer "F.Cu") (net 3))
-  (segment (start 189.326 57.8698) (end 183.3484 51.8922) (width 0.5) (layer "F.Cu") (net 3))
-  (segment (start 192.3076 57.8698) (end 189.326 57.8698) (width 0.5) (layer "F.Cu") (net 3))
-  (segment (start 197.53 56.55) (end 193.6774 56.55) (width 0.5) (layer "B.Cu") (net 3))
-  (segment (start 202.25 61.27) (end 197.53 56.55) (width 0.5) (layer "B.Cu") (net 3))
+  (segment (start 192.4024 55.275) (end 186.7312 55.275) (width 0.5) (layer "F.Cu") (net 3))
+  (segment (start 192.4074 55.28) (end 192.4024 55.275) (width 0.5) (layer "F.Cu") (net 3))
+  (segment (start 186.7312 55.275) (end 183.3484 51.8922) (width 0.5) (layer "F.Cu") (net 3))
+  (segment (start 196.26 55.28) (end 192.4074 55.28) (width 0.5) (layer "B.Cu") (net 3))
+  (segment (start 202.25 61.27) (end 196.26 55.28) (width 0.5) (layer "B.Cu") (net 3))
   (segment (start 177.56 81.683456) (end 177.56 85.021532) (width 0.5) (layer "F.Cu") (net 4))
   (segment (start 202.25 82.27) (end 199.21 82.27) (width 0.5) (layer "F.Cu") (net 4))
@@
   (segment (start 191.465 85.31) (end 188.088 85.31) (width 0.5) (layer "B.Cu") (net 5))
   (segment (start 180.795 121.15) (end 183.5 118.445) (width 0.5) (layer "B.Cu") (net 5))
-  (segment (start 192.7774 51.8) (end 192.7774 54.91) (width 0.5) (layer "F.Cu") (net 6))
-  (segment (start 192.7774 54.91) (end 192.4074 55.28) (width 0.5) (layer "F.Cu") (net 6))
+  (segment (start 193.6774 56.55) (end 193.6274 56.55) (width 0.5) (layer "F.Cu") (net 6))
   (segment (start 185.8555 98.708125) (end 184.462375 97.315) (width 0.5) (layer "F.Cu") (net 7))
   (segment (start 179.5526 97.315) (end 177.27336 95.03576) (width 0.5) (layer "F.Cu") (net 7))
@@
   (segment (start 191.465 91.39) (end 190.11 91.39) (width 0.5) (layer "F.Cu") (net 22))
   (segment (start 190.11 91.39) (end 188.415 89.695) (width 0.5) (layer "F.Cu") (net 22))
-  (segment (start 184.8082 48.4432) (end 183.5582 47.1932) (width 0.5) (layer "B.Cu") (net 23))
-  (segment (start 187.7706 48.4432) (end 184.8082 48.4432) (width 0.5) (layer "B.Cu") (net 23))
   (segment (start 194.5818 70.8118) (end 194.5818 62.4078) (width 0.5) (layer "B.Cu") (net 23))
-  (segment (start 190.7972 56.2098) (end 190.7972 51.4698) (width 0.5) (layer "B.Cu") (net 23))
   (segment (start 191.1374 58.9634) (end 191.1374 56.55) (width 0.5) (layer "B.Cu") (net 23))
   (segment (start 194.5818 62.4078) (end 191.1374 58.9634) (width 0.5) (layer "B.Cu") (net 23))
+  (segment (start 191.1374 51.81) (end 187.7706 48.4432) (width 0.5) (layer "B.Cu") (net 23))
+  (segment (start 184.8082 48.4432) (end 183.5582 47.1932) (width 0.5) (layer "B.Cu") (net 23))
   (segment (start 199.085 75.315) (end 194.5818 70.8118) (width 0.5) (layer "B.Cu") (net 23))
-  (segment (start 190.7972 51.4698) (end 187.7706 48.4432) (width 0.5) (layer "B.Cu") (net 23))
-  (segment (start 191.1374 56.55) (end 190.7972 56.2098) (width 0.5) (layer "B.Cu") (net 23))
+  (segment (start 191.1374 56.55) (end 191.1374 51.81) (width 0.5) (layer "B.Cu") (net 23))
+  (segment (start 187.7706 48.4432) (end 184.8082 48.4432) (width 0.5) (layer "B.Cu") (net 23))
   (segment (start 177.56 68.331152) (end 173.278076 68.331152) (width 0.5) (layer "F.Cu") (net 24))
   (segment (start 177.56 68.331152) (end 178.556152 67.335) (width 0.5) (layer "F.Cu") (net 24))

Commit message: Rev. 2
Parts:
- added G***: Rev2, Triglav_Modular:Rev2, B.Cu at (148.5, 136.7)
- added G***: Rev2, Triglav_Modular:Rev2, B.Cu at (177.5, 151.9)
- added G***: Rev2, Triglav_Modular:Rev2, B.Cu at (174.2, 109.7)
- C2: value 15uF -> 15u
- D3, D4: value 1N5819 -> 1N5817
- U2, U3: value TL084* -> RC4136
- moved C8 26.7 mm to (197.8, 98.2), turned to 180 degrees
- moved C6 24.3 mm to (196.7, 71.9), turned to 180 degrees
- moved R38 21.5 mm to (195.3, 108.3), turned to 180 degrees
- moved C9 16.9 mm to (177.4, 105.0), turned to 180 degrees
- moved C5 16.7 mm to (177.4, 78.3), turned to 180 degrees
- moved R43 11.8 mm to (185.1, 108.3)
- moved R33 11.5 mm to (185.1, 83.9)
- moved G*** 10.0 mm to (152.7, 110.2)
- moved G*** 10.0 mm to (144.4, 135.0)
- moved G*** 10.0 mm to (142.9, 104.5)
- moved J1 10.0 mm to (134.5, 123.4)
- moved J2 10.0 mm to (134.2, 146.1)
- moved J3 10.0 mm to (154.6, 146.1)
- moved J5 10.0 mm to (162.4, 112.2)
- moved REF** 10.0 mm to (144.4, 57.9)
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Connections:
- C1 pad 2: GND -> P_GND
- C10 pad 2: GND -> P_GND
- C11 pad 1: GND -> P_GND
- C4 pad 1: GND -> P_GND
- C5 pad 2: GND -> P_GND
- C6 pad 1: GND -> P_GND
- C7 pad 2: GND -> P_GND
- C8 pad 1: GND -> P_GND
- C9 pad 2: GND -> P_GND
- J4 pad 3: GND -> P_GND
- J4 pad 4: GND -> P_GND
- J4 pad 5: GND -> P_GND
- J4 pad 6: GND -> P_GND
- J4 pad 7: GND -> P_GND
- J4 pad 8: GND -> P_GND
- J6 pad 2: GND -> P_GND
- Q5 pad 2: GND -> P_GND
- Q6 pad 1: GND -> P_GND
- R19 pad 2: GND -> P_GND
- R21 pad 2: GND -> P_GND
- R36 pad 2: GND -> P_GND
- R47 pad 2: GND -> P_GND
- RX3 pad 1: GND -> P_GND
- RX32 pad 1: GND -> P_GND
- RX52 pad 1: GND -> P_GND
- U2 pad 1: Net-(R27-Pad1) -> Net-(U2A--)
- U2 pad 10: /GND2 -> Net-(D1-A)
- U2 pad 11: -12V -> +12V
- U2 pad 12: Net-(U2D-+) -> Net-(R20-Pad2)
- U2 pad 13: Net-(U2D--) -> Net-(U2D-+)
- U2 pad 14: Net-(R20-Pad2) -> Net-(U2D--)
- U2 pad 2: Net-(U2A--) -> /GND2
- U2 pad 3: /GND2 -> Net-(R27-Pad1)
- U2 pad 4: +12V -> Net-(R32-Pad1)
- U2 pad 7: Net-(R32-Pad1) -> -12V
- U2 pad 8: Net-(D1-A) -> Net-(D1-K)
- U2 pad 9: Net-(D1-K) -> /GND2
- U3 pad 1: Net-(R44-Pad1) -> Net-(U3A--)
- U3 pad 10: /GND3 -> Net-(R39-Pad2)
- U3 pad 11: -12V -> +12V
- U3 pad 12: /GND2 -> Net-(R34-Pad1)
- U3 pad 13: Net-(U3D--) -> /GND2
- U3 pad 14: Net-(R34-Pad1) -> Net-(U3D--)
- U3 pad 2: Net-(U3A--) -> /GND3
- U3 pad 3: /GND3 -> Net-(R44-Pad1)
- U3 pad 4: +12V -> Net-(R42-Pad1)
- U3 pad 7: Net-(R42-Pad1) -> -12V
- U3 pad 8: Net-(R39-Pad2) -> Net-(U3C--)
- U3 pad 9: Net-(U3C--) -> /GND3
- VR1 pad 3: GND -> P_GND
Routing:
- net Net-(U3B--): track 21.1 -> 43.2 mm
- net Net-(U2B--): track 19.9 -> 37.8 mm
- net Net-(D1-K): track 63.6 -> 72.4 mm, vias 0 -> 1
- net Net-(U3C--): track 33.0 -> 25.0 mm
- net Net-(R20-Pad2): track 91.6 -> 99.5 mm, vias 1 -> 0
- net Net-(D1-A): track 57.3 -> 64.0 mm, vias 4 -> 2
- net -12V: track 140.6 -> 146.4 mm
- net Net-(U3A--): track 34.6 -> 40.0 mm, vias 0 -> 1
- net Net-(U2A--): track 16.0 -> 21.0 mm
- net /GND3: track 30.5 -> 34.5 mm
- net Net-(Q5-E): track 9.33 -> 6.16 mm
- net Net-(U2D--): track 33.7 -> 31.0 mm
- net Net-(R1-Pad1): track 23.0 -> 20.5 mm
- net Net-(R39-Pad2): track 42.4 -> 43.6 mm
- net Net-(U2D-+): track 13.9 -> 15.0 mm
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- removed copper zone on B.Cu, net GND
- removed copper zone on F.Cu, net GND
Other:
- board size 90.5 x 108.9 mm -> 80.5 x 108.9 mm
- board text added: "HEADER ON THIS SIDE"
